File: hardware/elbsupply.sch (KiCad schematic (older format))
At the start: 101 parts, among them CON1 AVR-ISP-6, IC1 ATMEGA8-AI, P1 OUT_POS, P2 OUT_GND, P3 POWER_IN, Q1 KST2907A, Q2 KST2907A, Q3 IRLML6302, Q4 2N2222A, Q5 2N2222A, SW1 SW_L, SW2 SW_R, SW3 SW_OE, SW4 SW_MD, U1 MC34063, U2 TPS54331DDA, U3 LM324, U4 LM358, U5 TS78L05CS, U6 LM350T, U7 LM334

Commit message: fixed voltage DAC amplifier gain issue
Parts:
- removed R? (x2): 10k, symbol R
- Q3: symbol Q_PMOS_GSD -> Q_PMOS_GSD-RESCUE-elbsupply
- Q4, Q5: symbol Q_NPN_BEC -> Q_NPN_BEC-RESCUE-elbsupply
- RV1: symbol POT -> POT-RESCUE-elbsupply
- U3: symbol LM324 -> LM324-RESCUE-elbsupply
- U4: symbol LM358 -> LM358-RESCUE-elbsupply
Connections:
- wire segments 371 -> 367
Other:
- moved on the sheet: C21, C23, RP4
Changed lines of the file:
@@
 EESchema Schematic File Version 2
+LIBS:elbsupply-rescue
 LIBS:power
 LIBS:device
@@
 LIBS:memory
 LIBS:xilinx
-LIBS:special
 LIBS:microcontrollers
 LIBS:dsp
@@
 $EndComp
 $Comp
-L POT RV1
+L POT-RESCUE-elbsupply RV1
 U 1 1 54E38280
 P 10000 7350
@@
 L C C21
 U 1 1 54E561A9
-P 11050 5650
-F 0 "C21" H 11100 5750 50  0000 L CNN
-F 1 "1uF" H 11100 5550 50  0000 L CNN
-F 2 "Capacitors_SMD:C_0805_HandSoldering" H 11088 5500 30  0001 C CNN
-F 3 "" H 11050 5650 60  0000 C CNN
-	1    11050 5650
+P 11250 5700
+F 0 "C21" H 11300 5800 50  0000 L CNN
+F 1 "1uF" H 11300 5600 50  0000 L CNN
+F 2 "Capacitors_SMD:C_0805_HandSoldering" H 11288 5550 30  0001 C CNN
+F 3 "" H 11250 5700 60  0000 C CNN
+	1    11250 5700
 	-1   0    0    -1
 $EndComp
@@
 L GND #PWR013
 U 1 1 54E5E974
-P 11450 5900
-F 0 "#PWR013" H 11450 5650 60  0001 C CNN
-F 1 "GND" H 11450 5750 60  0000 C CNN
-F 2 "" H 11450 5900 60  0000 C CNN
-F 3 "" H 11450 5900 60  0000 C CNN
-	1    11450 5900
+P 11800 5950
+F 0 "#PWR013" H 11800 5700 60  0001 C CNN
+F 1 "GND" H 11800 5800 60  0000 C CNN
+F 2 "" H 11800 5950 60  0000 C CNN
+F 3 "" H 11800 5950 60  0000 C CNN
+	1    11800 5950
 	-1   0    0    -1
 $EndComp
@@
 L GND #PWR014
 U 1 1 54E5EB36
-P 11050 5900
-F 0 "#PWR014" H 11050 5650 60  0001 C CNN
-F 1 "GND" H 11050 5750 60  0000 C CNN
-F 2 "" H 11050 5900 60  0000 C CNN
-F 3 "" H 11050 5900 60  0000 C CNN
-	1    11050 5900
+P 11250 5950
+F 0 "#PWR014" H 11250 5700 60  0001 C CNN
+F 1 "GND" H 11250 5800 60  0000 C CNN
+F 2 "" H 11250 5950 60  0000 C CNN
+F 3 "" H 11250 5950 60  0000 C CNN
+	1    11250 5950
 	-1   0    0    -1
 $EndComp
@@
 Text Label 5800 4850 0    60   ~ 0
 I_PWM
-Text Label 10350 5450 0    60   ~ 0
+Text Label 10800 5450 0    60   ~ 0
 V_PWM
 Text Label 8900 5600 2    60   ~ 0
@@
 Constant current\nLED backlight driver\nI = 0.7V / 10R = 70mA
 $Comp
-L Q_PMOS_GSD Q3
+L Q_PMOS_GSD-RESCUE-elbsupply Q3
 U 1 1 55381159
 P 9150 10450
@@
 NoConn ~ 11500 2300
 $Comp
-L Q_NPN_BEC Q4
+L Q_NPN_BEC-RESCUE-elbsupply Q4
 U 1 1 5539C28E
 P 10600 3450
@@
 $EndComp
 $Comp
-L Q_NPN_BEC Q5
+L Q_NPN_BEC-RESCUE-elbsupply Q5
 U 1 1 5539C627
 P 11750 9500
@@
 $EndComp
 $Comp
-L LM324 U3
+L LM324-RESCUE-elbsupply U3
 U 1 1 55380929
 P 7150 3350
@@
 $EndComp
 $Comp
-L LM324 U3
+L LM324-RESCUE-elbsupply U3
 U 3 1 55380D0A
 P 9400 3450
@@
 $EndComp
 $Comp
-L LM324 U3
+L LM324-RESCUE-elbsupply U3
 U 4 1 55381002
 P 11950 3450
@@
 $EndComp
 $Comp
-L LM324 U3
+L LM324-RESCUE-elbsupply U3
 U 2 1 55381403
 P 7500 1900
@@
 L R_PACK4 RP4
 U 1 1 5538E9E3
-P 11700 5500
-F 0 "RP4" H 11700 5950 50  0000 C CNN
-F 1 "10k" H 11700 6050 50  0000 C CNN
-F 2 "devthrash:YC164-Yageo-Handsoldering" H 11700 5500 60  0001 C CNN
-F 3 "" H 11700 5500 60  0000 C CNN
-	1    11700 5500
+P 11550 5500
+F 0 "RP4" H 11550 5950 50  0000 C CNN
+F 1 "10k" H 11550 6050 50  0000 C CNN
+F 2 "devthrash:YC164-Yageo-Handsoldering" H 11550 5500 60  0001 C CNN
+F 3 "" H 11550 5500 60  0000 C CNN
+	1    11550 5500
 	-1   0    0    -1
 $EndComp
@@
 Voltage measurement\nvoltage divider\nRatio: 1/6
 $Comp
-L LM358 U4
+L LM358-RESCUE-elbsupply U4
 U 2 1 553A35B1
 P 12750 5350
@@
 $EndComp
 $Comp
-L LM358 U4
+L LM358-RESCUE-elbsupply U4
 U 1 1 553A38F1
 P 8300 4950
@@
 L C C23
 U 1 1 54E56232
-P 11450 5650
-F 0 "C23" H 11500 5750 50  0000 L CNN
-F 1 "1uF" H 11500 5550 50  0000 L CNN
-F 2 "Capacitors_SMD:C_0805_HandSoldering" H 11488 5500 30  0001 C CNN
-F 3 "" H 11450 5650 60  0000 C CNN
-	1    11450 5650
+P 11800 5700
+F 0 "C23" H 11850 5800 50  0000 L CNN
+F 1 "1uF" H 11850 5600 50  0000 L CNN
+F 2 "Capacitors_SMD:C_0805_HandSoldering" H 11838 5550 30  0001 C CNN
+F 3 "" H 11800 5700 60  0000 C CNN
+	1    11800 5700
 	1    0    0    -1
 $EndComp
@@
 	7400 5300 7400 5450
 Wire Wire Line
-	11050 5900 11050 5800
+	11250 5950 11250 5850
 Wire Wire Line
 	8200 8200 7850 8200
@@
 	1850 6100 1550 6100
 Wire Wire Line
-	11450 5900 11450 5800
+	11800 5950 11800 5850
 Connection ~ 15400 3800
 Wire Wire Line
@@
 	12150 5450 12250 5450
 Wire Wire Line
-	11500 5250 11400 5250
+	11350 5250 11250 5250
 Wire Wire Line
-	11400 5350 11500 5350
+	11250 5350 11350 5350
 Wire Wire Line
-	12250 5250 11900 5250
+	11750 5250 12250 5250
 Wire Wire Line
-	11400 4600 11400 5150
+	11250 4600 11250 5150
 Wire Wire Line
-	11400 5150 11500 5150
+	11250 5150 11350 5150
 Wire Wire Line
-	11900 5150 12000 5150
+	11750 5150 11850 5150
 Wire Wire Line
-	12000 5150 12000 5250
-Connection ~ 12000 5250
+	11850 5150 11850 5250
+Connection ~ 11850 5250
 Wire Wire Line
-	11400 4600 13350 4600
+	11250 4600 13350 4600
 Wire Wire Line
-	11900 5350 11950 5350
+	11750 5350 11800 5350
 Wire Wire Line
-	11950 5450 11900 5450
+	11800 5450 11750 5450
 $Comp
 L R_PACK4 RP6
@@
 	1    0    0    -1
 $EndComp
-$Comp
-L R R?
-U 1 1 5569D635
-P 10850 5450
-F 0 "R?" V 10930 5450 50  0000 C CNN
-F 1 "10k" V 10850 5450 50  0000 C CNN
-F 2 "" V 10780 5450 30  0000 C CNN
-F 3 "" H 10850 5450 30  0000 C CNN
-	1    10850 5450
-	0    -1   -1   0
-$EndComp
-$Comp
-L R R?
-U 1 1 5569DE11
-P 11250 5450
-F 0 "R?" V 11330 5450 50  0000 C CNN
-F 1 "10k" V 11250 5450 50  0000 C CNN
-F 2 "" V 11180 5450 30  0000 C CNN
-F 3 "" H 11250 5450 30  0000 C CNN
-	1    11250 5450
-	0    -1   -1   0
-$EndComp
-Wire Wire Line
-	11400 5250 11400 5350
-Wire Wire Line
-	11950 5350 11950 5450
-Wire Wire Line
-	11500 5450 11400 5450
-Wire Wire Line
-	11450 5450 11450 5500
-Connection ~ 11450 5450
 Wire Wire Line
-	11050 5500 11050 5450
+	11250 5250 11250 5550
 Wire Wire Line
-	11000 5450 11100 5450
-Connection ~ 11050 5450
+	11800 5350 11800 5550
 Wire Wire Line
-	10350 5450 10700 5450
+	10800 5450 11350 5450
 $Comp
 L VEE #PWR?
@@
 	-1   0    0    1
 $EndComp
+Connection ~ 11800 5450
+Connection ~ 11250 5350
 $EndSCHEMATC
